File: V0_Display/KiCad/V0_Display.sch (KiCad schematic (older format))
At the start: 28 parts, among them J1 USB_B_Micro, J2 I2C Header 1, J3 Conn_01x03, J4 Conn_01x02, J5 SWD Header, J7 USB_Header, J8 Conn_01x02, SW5 SW_SPST, SW6 SW_SPST, SW7 Rotary_Encoder_Switch, U1 AP2127K-3.3, U2 STM32F042F6Px, U3 74LVC1G17

Commit message: Create Atmega328p version of the V0 Display
Parts:
- removed C1, C2: 4.7uF, V0-Display:C_0805_2012Metric, symbol Device:C
- removed J3: Conn_01x03, V0-Display:PinHeader_1x03_P2.54mm_Vertical, symbol V0_Display:Conn_01x03
- removed J4: Conn_01x02, V0-Display:PinHeader_1x02_P2.54mm_Vertical, symbol V0_Display:Conn_01x02
- removed J5: SWD Header, V0-Display:PinHeader_2x05_P1.27mm_Vertical_SMD, symbol V0_Display:Conn_02x05_Odd_Even
- removed R2: 10K, V0-Display:R_0805_2012Metric, symbol V0_Display:R
- removed U1: AP2127K-3.3, V0-Display:SOT-23-5, symbol V0_Display:AP2127K-3.3
- removed U2: STM32F042F6Px, V0-Display:TSSOP-20_4.4x6.5mm_P0.65mm, symbol V0_Display:STM32F042F6Px
- removed U3: 74LVC1G17, V0-Display:SOT-753, symbol V0_Display:74LVC1G17
- added C1, C10, C11, C2, C9: 0.1uF, V0-Display:C_0603_1608Metric, symbol V0_Display:C
- added C5, C6, C7, C8: 22pF, V0-Display:C_0603_1608Metric, symbol Device:C_Small
- added D2: 5819, V0-Display:D_SOD-123, symbol Device:D_Schottky
- added J3: ICSP, V0-Display:PinHeader_2x03_P2.54mm_Vertical, symbol Connector_Generic:Conn_02x03_Odd_Even
- added R4: 1K, V0-Display:R_0805_2012Metric, symbol V0_Display:R
- added U4: ATmega328P-AU, V0-Display:TQFP-32_7x7mm_P0.8mm, symbol MCU_Microchip_ATmega:ATmega328P-AU
- added U5: CH340G, V0-Display:SOIC-16_3.9x9.9mm_P1.27mm, symbol Interface_USB:CH340G
- added Y1: 12MHz, V0-Display:Crystal_SMD_3225-4Pin_3.2x2.5mm, symbol Device:Crystal_GND24_Small
- added Y2: 16MHz, V0-Display:Crystal_SMD_3225-4Pin_3.2x2.5mm, symbol Device:Crystal_GND24_Small
- C3, C4: footprint V0-Display:C_0805_2012Metric -> V0-Display:C_0603_1608Metric; LCSC C49678 -> C14663
- R3: value 10K -> 1K; LCSC C17414 -> C17513
Connections:
- net labels added: +5V, MISO, MOSI, RXD, SCK, TXD
- net labels removed: +3V3, BOOT0, GPIO4, SWDCLK, SWDIO
- wire segments 86 -> 99
- no-connect marks 4 -> 0
Other:
- moved on the sheet: C3, C4, GPIO1, J2, J7, JP1, JP2, R1, SW5, SW6, SW7
