File: Daylight/Daylight.kicad_pcb (KiCad board)
At the start: 2 copper layers, 270 x 11 mm, 30 parts, among them J1 Conn_01x02_Female, J2 Conn_01x02_Female

Commit message: Flipped leds for DFH
Parts:
- D1, D10, D11, D12, D13, D14, D15, D16, D17, D18, D2, D3, D4, D5, D6, D7, D8, D9: footprint Daylight:LED_PLCC_2835_Handsoldering -> Daylight:LED_PLCC_2835_Handsoldering_flipped
Connections:
- H1 pad 1: GND -> unconnected-(H1-Pad1)
- H2 pad 1: GND -> unconnected-(H2-Pad1)
Other:
- board text added: "Daylight on a stick v1.2f by Blamm"
- board text removed: "Daylight on a stick v1.1 by Blamm"
